File: Electronic-Load-XY-FZ25_ESP32C3-Circuit/Electronic-Load-XY-FZ25_ESP32C3-Circuit.kicad_pcb (KiCad board)
At the start: 2 copper layers, 91 x 31 mm, 19 parts, among them IC1 BD5330G, J1 Banana-Socket, J10 Conn_Terminal-Block_1x2, J2 Banana-Socket, J3 mech.-solder-pad_large, J4 mech.-solder-pad_large, J5 Conn_1x2_PH, J6 Conn_1x2_PH, J7 Conn_1x3_PH, J8 mech.-solder-pad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

Commit message: Add v2.0 Circuit and footprint
Parts:
- removed D1: SBR2U30P1-7, Marcus-PCB-Library:SODFL3718X100N
- removed J5, J6: Conn_1x2_PH, Marcus-PCB-Library:Mechc.-solder-pad_1x2
- removed J7: Conn_1x3_PH, Marcus-PCB-Library:Mechc.-solder-pad_1x3
- removed Q1: AO3415, Package_TO_SOT_SMD:SOT-23
- added 3.3V: Conn_1x3_PH, Marcus-PCB-Library:Mechc.-solder-pad_1x3, F.Cu at (69.4, 69.4)
- added 5.1V: Conn_1x3_PH, Marcus-PCB-Library:Mechc.-solder-pad_1x3, F.Cu at (97.3, 69.4)
- added B+: Conn_1x2_PH, Marcus-PCB-Library:Mechc.-solder-pad_1x2, F.Cu at (72.2, 69.4)
- added Q2: AO3416, Package_TO_SOT_SMD:SOT-23, F.Cu at (66.8, 61.6)
- added SW: Conn_1x2_PH, Marcus-PCB-Library:Mechc.-solder-pad_1x2, F.Cu at (79.2, 69.4)
- J9: footprint Marcus-PCB-Library:Conn_1x4_PH -> Marcus-PCB-Library:Conn_1x4_PH_drill dot
- R3: footprint Resistor_SMD:R_1206_3216Metric -> Resistor_SMD:R_1206_3216Metric_Pad1.30x1.75mm_HandSolder
- U1: footprint Marcus-PCB-Library:TP5000-Charge-IC -> Marcus-PCB-Library:TP5000-Charge-IC_smal-led
- moved R3 28.5 mm to (107.2, 52.6), turned to -90 degrees
- moved IC1 7.48 mm to (66.8, 56.5), turned to -90 degrees
- moved J8 6.45 mm to (88.1, 70.3), turned to 90 degrees
- moved R2 4.95 mm to (69.8, 48.8), turned to -90 degrees
- moved R1 2.45 mm to (69.8, 44.9)
- moved U3 1.73 mm to (72.6, 60.9)
Connections:
- net Net-(U2-VBus) renamed Banana+
- net Net-(U2-Vin-) renamed L+
- IC1 pad 2: Net-(IC1-VDD) -> V-BATT+
- IC1 pad 3: GND -> Net-(IC1-GND)
- R3 pad 1: +5V -> Net-(U3-5V)
- R3 pad 2: Net-(U3-5V) -> +5V
Routing:
- net +3.3V: track 46.9 -> 104.0 mm
- net +5V: track 37.9 -> 14.7 mm
- net V-BATT+: track 62.1 -> 84.2 mm
- net Net-(IC1-GND): track 0.00 -> 18.5 mm
- net Net-(U3-5V): track 36.8 -> 18.4 mm
- net GND: track 129.0 -> 112.0 mm, vias 3 -> 2
- net Net-(IC1-VDD): track 9.31 -> 0.00 mm
- net Net-(J9-SCK): track 69.8 -> 61.6 mm
- net Net-(U3-PA02_A0_D0): track 4.84 -> 10.6 mm
- net Net-(J9-SDA): track 73.6 -> 68.2 mm
- net Net-(J6-V+): track 5.20 -> 0.00 mm
- net Banana+: track 66.8 -> 62.6 mm
- net Net-(J7-5.1V_out): track 8.01 -> 3.89 mm
- net Net-(J6-B+): track 0.00 -> 3.70 mm
- net Net-(IC1-VOUT): track 4.16 -> 6.73 mm
- added copper zone on F.Cu, net Banana+
- added copper zone on F.Cu, net L+
Other:
- board text added: "G"
- board text added: "V+"
- board text removed: "B+"
- board text removed: "FZ25 V+"
- board text removed: "GND"
- board text removed: "OUT+"
